File: PCB/ultraterm/ultraterm-nobites.kicad_pcb (KiCad board)
At the start: 2 copper layers, 73.1 x 78 mm, 18 parts, among them J1 ILI9341, J2 Battery_plug, J3 SD_Card_Receptacle, J4 SD_Card_Device, J5 Micro_SD_Card, SW1 SW_Push, SW2 SW_Push, SW3 SW_Push, SW4 SW_SPST, U1 XIAO-ESP32-S3-SMD, U2 LM809

Commit message: fiddled with PCB for export
Parts:
- removed mouse-bite-3mm-slot (x3): VAL**, Panelization:mouse-bite-3mm-slot
Routing:
- net GND: vias 11 -> 10
Other:
- outline, holes or cut-outs redrawn
