File: PCB/ultraterm/ultraterm.kicad_pcb (KiCad board)
At the start: 2 copper layers, 73.1 x 78 mm, 18 parts, among them J1 ILI9341, J2 Battery_plug, J3 SD_Card_Receptacle, J4 SD_Card_Device, J5 Micro_SD_Card, SW1 SW_Push, SW2 SW_Push, SW3 SW_Push, SW4 SW_SPST, U1 XIAO-ESP32-S3-SMD, U2 LM809

Commit message: Revised for TINYPICO
Parts:
- removed U1: XIAO-ESP32-S3-SMD, XAIO:XIAO-ESP32S3-SMD
- added LED1: LED_5mm_RGB_Kcom_RKGB, PCM_LED_THT_AKL:LED_D5.0mm-4_RGB_Wide_Pins, F.Cu at (113.2, 117.3)
- added R1: 33ohm, Resistor_THT:R_Axial_DIN0207_L6.3mm_D2.5mm_P10.16mm_Horizontal, F.Cu at (115.6, 137.1)
- added U3: ~, RF_Module:TINYPICO, F.Cu at (102.6, 141.4)
- J3: footprint Connector_Card:SD_Kyocera_145638009511859+ -> XAIO:AMPHENOL_10067847-001RLF
- SW4: footprint Button_Switch_THT:SW_PUSH_6mm_H13mm -> Button_Switch_THT:SW_Slide_SPDT_Angled_CK_OS102011MA1Q
- moved SW4 25.6 mm to (123.2, 134.2), turned to 90 degrees
- moved REF** 23.2 mm to (98.9, 119.7), turned to -90 degrees
- moved J3 11.9 mm to (76.0, 144.1)
- moved J2 11.0 mm to (119.4, 118.5), turned to 180 degrees
Connections:
- net Net-(J1-CLK) renamed CLK
- J2 pad 2: Net-(J2-Pin_2) -> VBAT
- SW4 pad 2: Net-(SW4-B) -> GND
Routing:
- net VBAT: track 0.00 -> 51.0 mm
- net +3V3: track 58.7 -> 99.8 mm, vias 1 -> 0
- net MISO: track 109.6 -> 142.9 mm, vias 2 -> 0
- net MOSI: track 100.8 -> 132.3 mm, vias 1 -> 0
- net SD CS: track 41.4 -> 14.7 mm, vias 2 -> 0
- net Net-(SW4-B): track 24.8 -> 0.00 mm, vias 1 -> 0
- net LED_R: track 0.00 -> 22.1 mm
- net Net-(J2-Pin_2): track 20.1 -> 0.00 mm
- net LCD_DS: track 45.1 -> 26.2 mm
- net CLK: track 89.1 -> 104.8 mm, vias 2 -> 1
- net LCD_CS: track 38.3 -> 23.6 mm
- net b2: track 50.2 -> 60.2 mm
- net b1: track 29.7 -> 38.2 mm
- net Net-(LED1-A): track 0.00 -> 8.39 mm
- net GND: track 81.1 -> 73.3 mm, vias 11 -> 6
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
Commit message: IO seems good?
Parts:
- moved J2 50.0 mm to (118.6, 68.5)
- moved J3 50.0 mm to (75.2, 94.1)
- moved R1 50.0 mm to (114.8, 87.1)
- moved REF** 50.0 mm to (114.5, 60.2)
- moved SW2 50.0 mm to (80.7, 53.2)
- moved mouse-bite-3mm-slot 50.0 mm to (119.0, 41.3)
- moved J1 50.0 mm to (125.0, 54.9)
- moved J4 50.0 mm to (91.9, 34.2)
- moved J5 50.0 mm to (110.2, 32.1)
- moved REF** 50.0 mm to (72.0, 55.7)
- moved REF** 50.0 mm to (93.4, 55.7)
- moved SW1 50.0 mm to (102.2, 53.2)
- moved SW3 50.0 mm to (59.5, 53.2)
- moved mouse-bite-3mm-slot 50.0 mm to (95.0, 47.7)
- moved mouse-bite-3mm-slot 50.0 mm to (119.0, 58.3)
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
Commit message: Final beta firmware.
Parts:
- moved J2 38.4 mm to (134.2, 103.6)
- moved REF** 38.4 mm to (130.1, 95.3)
- moved mouse-bite-3mm-slot 38.4 mm to (134.6, 76.3)
- moved J3 38.4 mm to (90.9, 129.2)
- moved J4 38.4 mm to (107.5, 69.2)
- moved R1 38.4 mm to (130.4, 122.1)
- moved SW2 38.4 mm to (96.4, 88.2)
- moved mouse-bite-3mm-slot 38.4 mm to (134.6, 93.3)
- moved J1 38.4 mm to (140.6, 89.9)
- moved J5 38.4 mm to (125.8, 67.2)
- moved REF** 38.4 mm to (87.6, 90.7)
- moved REF** 38.4 mm to (109.0, 90.7)
- moved SW1 38.4 mm to (117.9, 88.2)
- moved SW3 38.4 mm to (75.1, 88.2)
- moved SW4 38.4 mm to (138.0, 119.3)
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