File: PCB/ultraterm/ultraterm.kicad_sch (KiCad schematic)
At the start: 11 parts, among them J1 ILI9341, J2 Battery_plug, J3 SD_Card_Receptacle, J4 SD_Card_Device, J5 Micro_SD_Card, SW1 SW_Push, SW2 SW_Push, SW3 SW_Push, SW4 SW_SPST, U1 XIAO-ESP32-S3-SMD, U2 LM809

Commit message: Revised for TINYPICO
Parts:
- removed U1: XIAO-ESP32-S3-SMD, XAIO:XIAO-ESP32S3-SMD, symbol Seeed_Studio_XIAO_Series:XIAO-ESP32-S3-SMD
- added LED1: LED_5mm_RGB_Kcom_RKGB, PCM_LED_THT_AKL:LED_D5.0mm-4_RGB_Wide_Pins, symbol PCM_LED_AKL:LED_5mm_RGB_Acom_RABG
- added R1: 33ohm, Resistor_THT:R_Axial_DIN0207_L6.3mm_D2.5mm_P10.16mm_Horizontal, symbol PCM_SL_Resistors:33ohm
- added U3: ~, RF_Module:TINYPICO, symbol MCU_Espressif:TINYPICO
Connections:
- net +3V3: now also R1.1, U3.14 (3v3)
- net GND: now also SW4.2 (B), U3.10 (GND), U3.12 (GND)
- net LCD_CS: now also U3.6 (21)
- net LCD_DS: now also U3.7 (32)
- net MISO: now also U3.2 (19)
- net MOSI: now also U3.3 (18)
- net SD CS: now also U3.19 (26)
- net TOUCH_CS: now also U3.4 (5)
- net TOUCH_PEN: now also U3.1 (23)
- net b1: now also U3.17 (15)
- net b2: now also U3.16 (17)
- net b3: now also U3.15 (4)
- net VBAT: now reaches J2.2 (Pin_2)
- net VBAT: now also U3.11 (VBAT)
- net CLK: now reaches J1.10 (CLK), J1.7 (SCK), J3.5 (CLK)
- net CLK: now also U3.5 (22)
- new net: LED1.2 (A), R1.2
- new net LED_B: LED1.4 (B), U3.8 (27)
- new net LED_G: LED1.3 (G), U3.9 (RES)
- new net LED_R: LED1.1 (R), U3.20 (25)
Other:
- moved on the sheet: J2, SW4

Commit message: Final beta firmware.
Other:
- moved on the sheet: J1, J2, J3, J4, J5, LED1, R1, SW1, SW2, SW3, SW4, U2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
